File: ser-if/rs232.brd (EAGLE design)
At the start: 100 x 80 mm, 19 parts, among them IC1 8251A, IC2 74LS93N, IC3 74LS00N, IC4 74LS245N, X1 MAC64L

Commit message: Add files via upload
Connections:
- net A4: now also 7485.15; no longer 7485.10
- net A5: now also 7485.13; no longer 7485.12
- net A6: now also 7485.12; no longer 7485.13
- net A7: now also 7485.10; no longer 7485.15
Routing:
- net N$27: track 87.0 -> 116.4 mm, vias 1 -> 0
- net N$7: track 159.4 -> 132.5 mm, vias 0 -> 1
- net A0: track 72.9 -> 49.0 mm, vias 0 -> 1
- net IOR: track 87.0 -> 104.2 mm
- net N$12: track 87.4 -> 73.2 mm
- net A7: track 49.8 -> 38.2 mm
- net A4: track 43.7 -> 32.1 mm
- net CLK: track 108.5 -> 117.4 mm
- net N$4: track 31.2 -> 22.9 mm
- net N$11: track 25.4 -> 19.0 mm
- net N$9: track 71.3 -> 65.6 mm, vias 0 -> 1
- net IOW: track 112.1 -> 106.5 mm, vias 1 -> 0
- net N$5: track 51.9 -> 46.6 mm, vias 1 -> 0
- net GND: track 291.1 -> 295.9 mm
- net N$6: track 37.7 -> 33.5 mm
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
Commit message: Add files via upload
Parts:
- added C5: 4,7u, rcl:E5-6
Connections:
- net N$1 renamed R1
- net N$12 renamed /CS
- net N$13 renamed TXD
- net N$14 renamed RXD
- net N$15 renamed DSR
- net N$16 renamed DTR
- net N$17 renamed CTS
- net N$18 renamed RTS
- net N$2 renamed R2
- net N$20 renamed -D7
- net N$21 renamed -D6
- net N$22 renamed -D5
- net N$23 renamed -D4
- net N$24 renamed -D3
- net N$25 renamed -D2
- net N$26 renamed -D1
- net N$27 renamed -CLK
- net N$28 renamed -D0
- net N$3 renamed R3
- net N$4 renamed R4
- net N$5 renamed -RES
- net N$7 renamed RTXC
- removed net VCC: IC4.20
- net +5V: now also C5.+, IC4.20
- net GND: now also C5.-
Routing:
- net +5V: track 233.4 -> 258.1 mm
- net GND: track 295.9 -> 301.6 mm
Other:
- board text added: "Serial Interface"
- board text added: "VzEkC"
Changed lines of the file:
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@@
 <wire x1="100" y1="80" x2="0" y2="80" width="0" layer="20"/>
 <wire x1="0" y1="80" x2="0" y2="0" width="0" layer="20"/>
+<text x="93.25" y="11.25" size="1.778" layer="1" rot="R90">VzEkC</text>
+<text x="96.75" y="11.5" size="1.778" layer="1" rot="R90">Serial Interface</text>
 </plain>
 <attributes>
@@
 <element name="C4" library="rcl" package="C025-025X050" value="100n" x="70.19" y="34.61" rot="R90"/>
 <element name="IC4" library="74xx-eu" package="DIL20" value="74LS245N" x="23.13" y="55.43"/>
+<element name="C5" library="rcl" package="E5-6" value="4,7u" x="10.5" y="16.75" rot="R90"/>
 </elements>
 <signals>
@@
 <wire x1="43" y1="54" x2="43.12" y2="53.78" width="0.254" layer="1"/>
 <wire x1="15.5" y1="25" x2="17" y2="26.5" width="0.254" layer="16"/>
-<wire x1="9" y1="25" x2="15.5" y2="25" width="0.254" layer="16"/>
+<wire x1="9" y1="25" x2="10.5" y2="25" width="0.254" layer="16"/>
+<wire x1="10.5" y1="25" x2="15.5" y2="25" width="0.254" layer="16"/>
 <wire x1="6.5" y1="27.5" x2="9" y2="25" width="0.254" layer="16"/>
 <wire x1="6.5" y1="33" x2="6.5" y2="27.5" width="0.254" layer="16"/>
@@
 <wire x1="43.5" y1="51" x2="43.12" y2="51.24" width="0.254" layer="16"/>
 <wire x1="70" y1="36" x2="70.19" y2="35.88" width="0.254" layer="16"/>
-</signal>
-<signal name="VCC">
-<contactref element="IC4" pad="20"/>
-</signal>
-<signal name="N$1">
+<contactref element="C5" pad="-"/>
+<wire x1="10.5" y1="25" x2="10.5" y2="19.29" width="0.254" layer="16"/>
+</signal>
+<signal name="R1">
 <contactref element="7485" pad="1"/>
 <contactref element="R1" pad="1"/>
@@
 <wire x1="51" y1="59" x2="50.74" y2="58.86" width="0.254" layer="16"/>
 </signal>
-<signal name="N$2">
+<signal name="R2">
 <contactref element="7485" pad="14"/>
 <contactref element="S1" pad="7"/>
@@
 <wire x1="55.5" y1="56.5" x2="55.62" y2="56.89" width="0.254" layer="16"/>
 </signal>
-<signal name="N$3">
+<signal name="R3">
 <contactref element="7485" pad="11"/>
 <contactref element="S1" pad="6"/>
@@
 <wire x1="50.5" y1="53.5" x2="50.74" y2="53.78" width="0.254" layer="16"/>
 </signal>
-<signal name="N$4">
+<signal name="R4">
 <contactref element="7485" pad="9"/>
 <contactref element="S1" pad="5"/>
@@
 <wire x1="14.5" y1="42" x2="14.52" y2="42.03" width="0.254" layer="16"/>
 <wire x1="10.5" y1="57" x2="7.44" y2="53.94" width="0.254" layer="1"/>
-<wire x1="10.5" y1="69.5" x2="10.5" y2="57" width="0.254" layer="1"/>
+<wire x1="10.5" y1="69.5" x2="10.5" y2="59.5" width="0.254" layer="1"/>
+<wire x1="10.5" y1="59.5" x2="10.5" y2="57" width="0.254" layer="1"/>
 <wire x1="10.5" y1="69.5" x2="10.83" y2="69.75" width="0.254" layer="1"/>
 <wire x1="11" y1="70" x2="11" y2="74.5" width="0.254" layer="1"/>
@@
 <wire x1="48.5" y1="39" x2="48.84" y2="38.74" width="0.254" layer="16"/>
 <wire x1="50" y1="36.5" x2="65.5" y2="36.5" width="0.254" layer="1"/>
+<contactref element="IC4" pad="20"/>
+<wire x1="10.5" y1="59.5" x2="11.5" y2="59.5" width="0.254" layer="1"/>
+<wire x1="11.5" y1="59.5" x2="11.7" y2="59.24" width="0.254" layer="1"/>
+<contactref element="C5" pad="+"/>
+<wire x1="6.5" y1="35.5" x2="7.5" y2="34.5" width="0.254" layer="1"/>
+<wire x1="6.5" y1="35.5" x2="6.06" y2="35.61" width="0.254" layer="1"/>
+<wire x1="7.5" y1="17.5" x2="10.5" y2="14.5" width="0.254" layer="1"/>
+<wire x1="7.5" y1="34.5" x2="7.5" y2="17.5" width="0.254" layer="1"/>
+<wire x1="10.5" y1="14.5" x2="10.5" y2="14.21" width="0.254" layer="1"/>
 </signal>
 <signal name="N$11">
@@
 <wire x1="61.5" y1="31" x2="61.54" y2="31.12" width="0.254" layer="1"/>
 </signal>
-<signal name="N$12">
+<signal name="/CS">
 <contactref element="7404" pad="2"/>
 <contactref element="IC1" pad="11"/>
@@
 <via x="47" y="28" extent="1-16" drill="0.6096"/>
 </signal>
-<signal name="N$27">
+<signal name="-CLK">
 <contactref element="7404" pad="6"/>
 <contactref element="IC1" pad="20"/>
@@
 <wire x1="13.5" y1="75" x2="13.37" y2="74.83" width="0.254" layer="1"/>
 </signal>
-<signal name="N$7">
+<signal name="RTXC">
 <contactref element="IC2" pad="11"/>
 <contactref element="IC1" pad="25"/>
@@
 <wire x1="89.5" y1="58" x2="89.69" y2="58.46" width="0.254" layer="16"/>
 </signal>
-<signal name="N$13">
+<signal name="TXD">
 <contactref element="JP1" pad="2"/>
 <contactref element="IC1" pad="19"/>
@@
 <wire x1="33" y1="8.5" x2="32.71" y2="8.46" width="0.254" layer="1"/>
 </signal>
-<signal name="N$15">
+<signal name="DSR">
 <contactref element="IC1" pad="22"/>
 <contactref element="JP1" pad="4"/>
@@
 <wire x1="27.5" y1="8.5" x2="27.63" y2="8.46" width="0.254" layer="1"/>
 </signal>
-<signal name="N$16">
+<signal name="DTR">
 <contactref element="IC1" pad="24"/>
 <contactref element="JP1" pad="5"/>
@@
 <via x="18.5" y="24.5" extent="1-16" drill="0.6096"/>
 </signal>
-<signal name="N$17">
+<signal name="CTS">
 <contactref element="IC1" pad="17"/>
 <contactref element="JP1" pad="6"/>
@@
 <via x="34" y="10.5" extent="1-16" drill="0.6096"/>
 </signal>
-<signal name="N$18">
+<signal name="RTS">
 <contactref element="IC1" pad="23"/>
 <contactref element="JP1" pad="7"/>
@@
 <wire x1="54" y1="31.5" x2="53.92" y2="31.12" width="0.254" layer="1"/>
 </signal>
-<signal name="N$14">
+<signal name="RXD">
 <contactref element="IC1" pad="3"/>
 <contactref element="JP1" pad="3"/>
@@
 <wire x1="30" y1="8" x2="30.17" y2="8.46" width="0.254" layer="1"/>
 </signal>
-<signal name="N$5">
+<signal name="-RES">
 <contactref element="7404" pad="4"/>
 <contactref element="IC1" pad="21"/>
@@
 <wire x1="59" y1="18.5" x2="59.14" y2="18.09" width="0.254" layer="16"/>
 </signal>
-<signal name="N$20">
+<signal name="-D7">
 <contactref element="IC1" pad="8"/>
 <contactref element="IC4" pad="2"/>
@@
 <via x="14" y="40" extent="1-16" drill="0.6096"/>
 </signal>
-<signal name="N$21">
+<signal name="-D6">
 <contactref element="IC1" pad="7"/>
 <contactref element="IC4" pad="3"/>
@@
 <wire x1="17" y1="52" x2="16.78" y2="51.62" width="0.254" layer="1"/>
 </signal>
-<signal name="N$22">
+<signal name="-D5">
 <contactref element="IC1" pad="6"/>
 <contactref element="IC4" pad="4"/>
@@
 <wire x1="19" y1="51.5" x2="19.32" y2="51.62" width="0.254" layer="1"/>
 </signal>
-<signal name="N$23">
+<signal name="-D4">
 <contactref element="IC1" pad="5"/>
 <contactref element="IC4" pad="5"/>
@@
 <wire x1="21.5" y1="51.5" x2="21.86" y2="51.62" width="0.254" layer="1"/>
 </signal>
-<signal name="N$24">
+<signal name="-D3">
 <contactref element="IC1" pad="2"/>
 <contactref element="IC4" pad="6"/>
@@
 <wire x1="24" y1="52" x2="24.4" y2="51.62" width="0.254" layer="1"/>
 </signal>
-<signal name="N$25">
+<signal name="-D2">
 <contactref element="IC1" pad="1"/>
 <contactref element="IC4" pad="7"/>
@@
 <wire x1="26.5" y1="52" x2="26.94" y2="51.62" width="0.254" layer="16"/>
 </signal>
-<signal name="N$26">
+<signal name="-D1">
 <contactref element="IC1" pad="28"/>
 <contactref element="IC4" pad="8"/>
@@
 <wire x1="29.5" y1="52" x2="29.48" y2="51.62" width="0.254" layer="16"/>
 </signal>
-<signal name="N$28">
+<signal name="-D0">
 <contactref element="IC1" pad="27"/>
 <contactref element="IC4" pad="9"/>

Commit message: Add files via upload
Parts:
- added R5, R6: 4k7, rcl:0207/10
- C5: device rcl:E5-6 -> rcl:E2,5-5
- moved JP1 4.00 mm to (26.4, 12.5)
- moved C5 2.30 mm to (11.0, 19.0), turned to 0 degrees
Connections:
- net DTR renamed /DTR
- net N$11 renamed A=B
- net N$6 renamed -A=B
- net RTS renamed /RTS
- removed net -RES: 7404.4, IC1.21
- removed net CTS: IC1.17, JP1.6
- removed net DSR: IC1.22, JP1.4
- new net /CTS: IC1.17, JP1.6, R6.2
- new net /DSR: IC1.22, JP1.4, R5.2
- new net /RES: 7404.3, X1.C13
- net GND: now also R5.1, R6.1
- net RES: now also 7404.4, IC1.21; no longer 7404.3, X1.C13
Routing:
- net /RES: track 0.00 -> 77.3 mm
- net /CTS: track 0.00 -> 51.2 mm
- net -RES: track 46.6 -> 0.00 mm
- net CTS: track 46.3 -> 0.00 mm, vias 1 -> 0
- net /DSR: track 0.00 -> 36.1 mm
- net DSR: track 35.0 -> 0.00 mm
- net +5V: track 258.1 -> 234.0 mm
- net IOR: track 104.2 -> 84.3 mm
- net -CLK: track 116.4 -> 96.6 mm
- net GND: track 301.6 -> 285.4 mm
- net /DTR: track 48.0 -> 32.1 mm
- net -D0: track 38.7 -> 24.3 mm
- net CLK: track 117.4 -> 105.9 mm
- net -D7: track 30.9 -> 42.3 mm, vias 1 -> 0
- net -D1: track 35.5 -> 24.2 mm
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