File: ser-if/rs232.sch (EAGLE design)
At the start: 19 parts, among them IC1 8251A, IC2 74LS93N, IC3 74LS00N, X1 MAC64L

Commit message: Add files via upload
Parts:
- removed 8255: 8255, micro-intel:8255A
- added IC4: 74LS245N, 74xx-eu:74LS245N
Connections:
- removed net N$20: IC3C.I0
- new net N$21: IC1.D7, IC4A.A1
- new net N$22: IC1.D6, IC4A.A2
- new net N$23: IC1.D5, IC4A.A3
- new net N$24: IC1.D4, IC4A.A4
- new net N$25: IC1.D3, IC4A.A5
- new net N$26: IC1.D2, IC4A.A6
- new net N$28: IC1.D1, IC4A.A7
- new net N$29: IC1.D0, IC4A.A8
- net +5V: no longer 8255P.VCC
- net A4: now also 7485A.A0; no longer 7485A.A3
- net A5: now also 7485A.A1; no longer 7485A.A2
- net A6: now also 7485A.A2; no longer 7485A.A1
- net A7: now also 7485A.A3; no longer 7485A.A0
- net D0: now also IC4A.B8; no longer IC1.D0
- net D1: now also IC4A.B7; no longer IC1.D1
- net D2: now also IC4A.B6; no longer IC1.D2
- net D3: now also IC4A.B5; no longer IC1.D3
- net D4: now also IC4A.B4; no longer IC1.D4
- net D5: now also IC4A.B3; no longer IC1.D5
- net D6: now also IC4A.B2; no longer IC1.D6
- net D7: now also IC4A.B1; no longer IC1.D7
- net GND: no longer 8255P.GND
- net IOR: now also IC3C.I0
- net IOW: now also IC4A.DIR
- net N$12: now also IC4A.G
- net N$14: no longer IC1.TXE, IC1.TXRDY
Other:
- moved on the sheet: 7404B, 7404D, 7404E, 7404F, 7404P, 7485P, C1, C2, C3, C4, H1, H2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

Commit message: Add files via upload
Connections:
- net A4: now also 7485A.A3; no longer 7485A.A0
- net A5: now also 7485A.A2; no longer 7485A.A1
- net A6: now also 7485A.A1; no longer 7485A.A2
- net A7: now also 7485A.A0; no longer 7485A.A3
Other:
- moved on the sheet: 7485, IC4

Commit message: Add files via upload
Parts:
- added C5: 4,7u, rcl:CPOL-EUE5-6
Connections:
- net N$1 renamed R1
- net N$12 renamed /CS
- net N$13 renamed TXD
- net N$14 renamed RXD
- net N$15 renamed DSR
- net N$16 renamed DTR
- net N$17 renamed CTS
- net N$18 renamed RTS
- net N$2 renamed R2
- net N$20 renamed -D7
- net N$21 renamed -D6
- net N$22 renamed -D5
- net N$23 renamed -D4
- net N$24 renamed -D3
- net N$25 renamed -D2
- net N$26 renamed -D1
- net N$27 renamed -CLK
- net N$28 renamed -D0
- net N$3 renamed R3
- net N$4 renamed R4
- net N$5 renamed -RES
- net N$7 renamed RTXC
- net +5V: now also C5.+, IC4P.VCC
- net GND: now also C5.-, IC4P.GND
Other:
- moved on the sheet: H1, H2
Changed lines of the file:
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@@
 <setting verticaltext="up"/>
 </settings>
-<grid distance="0.5" unitdist="mm" unit="mm" style="lines" multiple="1" display="no" altdistance="0.01" altunitdist="inch" altunit="inch"/>
+<grid distance="0.1" unitdist="inch" unit="inch" style="lines" multiple="1" display="no" altdistance="0.01" altunitdist="inch" altunit="inch"/>
 <layers>
 <layer number="1" name="Top" color="4" fill="1" visible="no" active="no"/>
@@
 <part name="C4" library="rcl" deviceset="C-EU" device="025-025X050" value="100n"/>
 <part name="IC4" library="74xx-eu" deviceset="74*245" device="N" technology="LS"/>
+<part name="P+9" library="supply1" deviceset="+5V" device=""/>
+<part name="GND9" library="supply1" deviceset="GND" device=""/>
+<part name="C5" library="rcl" deviceset="CPOL-EU" device="E5-6" value="4,7u"/>
 </parts>
 <sheets>
@@
 <instance part="GND7" gate="1" x="-60.96" y="-22.86"/>
 <instance part="GND8" gate="1" x="-71.12" y="-22.86"/>
-<instance part="H1" gate="G$1" x="-99.06" y="106.68"/>
-<instance part="H2" gate="G$1" x="-86.36" y="106.68"/>
+<instance part="H1" gate="G$1" x="-30.48" y="-22.86"/>
+<instance part="H2" gate="G$1" x="-17.78" y="-22.86"/>
 <instance part="GND10" gate="1" x="114.3" y="101.6" rot="R90"/>
 <instance part="GND11" gate="1" x="114.3" y="96.52" rot="R90"/>
@@
 <instance part="C4" gate="G$1" x="-43.18" y="111.76"/>
 <instance part="IC4" gate="A" x="68.58" y="7.62"/>
+<instance part="IC4" gate="P" x="-81.28" y="-12.7"/>
+<instance part="P+9" gate="1" x="-81.28" y="-2.54"/>
+<instance part="GND9" gate="1" x="-81.28" y="-22.86"/>
+<instance part="C5" gate="G$1" x="-81.28" y="111.76"/>
 </instances>
 <busses>
 </busses>
 <nets>
-<net name="N$1" class="0">
+<net name="R1" class="0">
 <segment>
 <wire x1="109.22" y1="91.44" x2="129.54" y2="91.44" width="0.1524" layer="91"/>
@@
 </segment>
 </net>
-<net name="N$2" class="0">
+<net name="R2" class="0">
 <segment>
 <wire x1="109.22" y1="88.9" x2="127" y2="88.9" width="0.1524" layer="91"/>
@@
 </segment>
 </net>
-<net name="N$3" class="0">
+<net name="R3" class="0">
 <segment>
 <wire x1="109.22" y1="86.36" x2="124.46" y2="86.36" width="0.1524" layer="91"/>
@@
 </segment>
 </net>
-<net name="N$4" class="0">
+<net name="R4" class="0">
 <segment>
 <wire x1="109.22" y1="83.82" x2="121.92" y2="83.82" width="0.1524" layer="91"/>
@@
 <junction x="-63.5" y="114.3"/>
 <junction x="-43.18" y="114.3"/>
-<junction x="-73.66" y="114.3"/>
+<pinref part="C5" gate="G$1" pin="+"/>
+<wire x1="-81.28" y1="114.3" x2="-73.66" y2="114.3" width="0.1524" layer="91"/>
 </segment>
 <segment>
@@
 <wire x1="-30.48" y1="35.56" x2="-25.4" y2="35.56" width="0.1524" layer="91"/>
 <wire x1="-30.48" y1="35.56" x2="-33.02" y2="35.56" width="0.1524" layer="91"/>
+</segment>
+<segment>
+<pinref part="IC4" gate="P" pin="VCC"/>
+<pinref part="P+9" gate="1" pin="+5V"/>
 </segment>
 </net>
@@
 <junction x="-63.5" y="106.68"/>
 <junction x="-43.18" y="106.68"/>
-<junction x="-73.66" y="106.68"/>
+<pinref part="C5" gate="G$1" pin="-"/>
+<wire x1="-81.28" y1="106.68" x2="-73.66" y2="106.68" width="0.1524" layer="91"/>
 </segment>
 <segment>
@@
 <wire x1="20.32" y1="48.26" x2="22.86" y2="48.26" width="0.1524" layer="91"/>
 </segment>
+<segment>
+<pinref part="IC4" gate="P" pin="GND"/>
+<pinref part="GND9" gate="1" pin="GND"/>
+</segment>
 </net>
 <net name="N$11" class="0">
@@
 </segment>
 </net>
-<net name="N$12" class="0">
+<net name="/CS" class="0">
 <segment>
 <wire x1="50.8" y1="99.06" x2="50.8" y2="88.9" width="0.1524" layer="91"/>
@@
 </segment>
 </net>
-<net name="N$27" class="0">
+<net name="-CLK" class="0">
 <segment>
 <pinref part="7404" gate="C" pin="O"/>
@@
 </segment>
 </net>
-<net name="N$7" class="0">
+<net name="RTXC" class="0">
 <segment>
 <pinref part="IC2" gate="A" pin="QD"/>
@@
 </segment>
 </net>
-<net name="N$13" class="0">
+<net name="TXD" class="0">
 <segment>
 <pinref part="JP1" gate="A" pin="2"/>
@@
 </segment>
 </net>
-<net name="N$15" class="0">
+<net name="DSR" class="0">
 <segment>
 <pinref part="IC1" gate="G$1" pin="!DSR"/>
@@
 </segment>
 </net>
-<net name="N$16" class="0">
+<net name="DTR" class="0">
 <segment>
 <pinref part="IC1" gate="G$1" pin="!DTR"/>
@@
 </segment>
 </net>
-<net name="N$17" class="0">
+<net name="CTS" class="0">
 <segment>
 <pinref part="IC1" gate="G$1" pin="!CTS"/>
@@
 </segment>
 </net>
-<net name="N$18" class="0">
+<net name="RTS" class="0">
 <segment>
 <pinref part="IC1" gate="G$1" pin="!RTS"/>
@@
 </segment>
 </net>
-<net name="N$14" class="0">
+<net name="RXD" class="0">
 <segment>
 <pinref part="IC1" gate="G$1" pin="RXD"/>
@@
 </segment>
 </net>
-<net name="N$5" class="0">
+<net name="-RES" class="0">
 <segment>
 <pinref part="7404" gate="B" pin="O"/>
@@
 </segment>
 </net>
-<net name="N$20" class="0">
+<net name="-D7" class="0">
 <segment>
 <pinref part="IC1" gate="G$1" pin="D7"/>
@@
 </segment>
 </net>
-<net name="N$21" class="0">
+<net name="-D6" class="0">
 <segment>
 <pinref part="IC1" gate="G$1" pin="D6"/>
@@
 </segment>
 </net>
-<net name="N$22" class="0">
+<net name="-D5" class="0">
 <segment>
 <pinref part="IC1" gate="G$1" pin="D5"/>
@@
 </segment>
 </net>
-<net name="N$23" class="0">
+<net name="-D4" class="0">
 <segment>
 <pinref part="IC1" gate="G$1" pin="D4"/>
@@
 </segment>
 </net>
-<net name="N$24" class="0">
+<net name="-D3" class="0">
 <segment>
 <pinref part="IC1" gate="G$1" pin="D3"/>
@@
 </segment>
 </net>
-<net name="N$25" class="0">
+<net name="-D2" class="0">
 <segment>
 <pinref part="IC1" gate="G$1" pin="D2"/>
@@
 </segment>
 </net>
-<net name="N$26" class="0">
+<net name="-D1" class="0">
 <segment>
 <pinref part="IC1" gate="G$1" pin="D1"/>
@@
 </segment>
 </net>
-<net name="N$28" class="0">
+<net name="-D0" class="0">
 <segment>
 <pinref part="IC1" gate="G$1" pin="D0"/>

Commit message: Add files via upload
Parts:
- added R5, R6: 4k7, rcl:R-EU_0207/10
- C5: device rcl:CPOL-EUE5-6 -> rcl:CPOL-EUE2.5-5
Connections:
- net DTR renamed /DTR
- net N$11 renamed A=B
- net N$6 renamed -A=B
- net RTS renamed /RTS
- removed net -RES: 7404B.O, IC1.RESET
- removed net CTS: IC1.!CTS, JP1.6
- removed net DSR: IC1.!DSR, JP1.4
- new net /CTS: IC1.!CTS, JP1.6, R6.2
- new net /DSR: IC1.!DSR, JP1.4, R5.2
- new net /RES: 7404B.I, X1.C13
- net GND: now also R5.1, R6.1
- net RES: now also 7404B.O, IC1.RESET; no longer 7404B.I, X1.C13
Other:
- moved on the sheet: C5
Changed lines of the file:
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@@
 <part name="P+9" library="supply1" deviceset="+5V" device=""/>
 <part name="GND9" library="supply1" deviceset="GND" device=""/>
-<part name="C5" library="rcl" deviceset="CPOL-EU" device="E5-6" value="4,7u"/>
+<part name="C5" library="rcl" deviceset="CPOL-EU" device="E2.5-5" value="4,7u"/>
+<part name="R5" library="rcl" deviceset="R-EU_" device="0207/10" value="4k7"/>
+<part name="R6" library="rcl" deviceset="R-EU_" device="0207/10" value="4k7"/>
 </parts>
 <sheets>
@@
 <instance part="GND19" gate="1" x="-86.36" y="60.96" rot="R270"/>
 <instance part="JP1" gate="A" x="-35.56" y="27.94" rot="R180"/>
-<instance part="GND20" gate="1" x="-33.02" y="10.16" rot="R270"/>
+<instance part="GND20" gate="1" x="-25.4" y="2.54"/>
 <instance part="P+12" gate="1" x="-35.56" y="43.18" rot="R90"/>
 <instance part="C3" gate="G$1" x="-73.66" y="111.76"/>
@@
 <instance part="P+9" gate="1" x="-81.28" y="-2.54"/>
 <instance part="GND9" gate="1" x="-81.28" y="-22.86"/>
-<instance part="C5" gate="G$1" x="-81.28" y="111.76"/>
+<instance part="C5" gate="G$1" x="-83.82" y="111.76"/>
+<instance part="R5" gate="G$1" x="-20.32" y="12.7" rot="R90"/>
+<instance part="R6" gate="G$1" x="-15.24" y="12.7" rot="R90"/>
 </instances>
 <busses>
@@
 <junction x="-63.5" y="114.3"/>
 <junction x="-43.18" y="114.3"/>
+<wire x1="-83.82" y1="114.3" x2="-73.66" y2="114.3" width="0.1524" layer="91"/>
 <pinref part="C5" gate="G$1" pin="+"/>
-<wire x1="-81.28" y1="114.3" x2="-73.66" y2="114.3" width="0.1524" layer="91"/>
 </segment>
 <segment>
@@
 <junction x="-63.5" y="106.68"/>
 <junction x="-43.18" y="106.68"/>
+<wire x1="-83.82" y1="106.68" x2="-73.66" y2="106.68" width="0.1524" layer="91"/>
 <pinref part="C5" gate="G$1" pin="-"/>
-<wire x1="-81.28" y1="106.68" x2="-73.66" y2="106.68" width="0.1524" layer="91"/>
 </segment>
 <segment>
@@
 <segment>
 <pinref part="GND20" gate="1" pin="GND"/>
-<wire x1="-30.48" y1="10.16" x2="-25.4" y2="10.16" width="0.1524" layer="91"/>
-<wire x1="-25.4" y1="10.16" x2="-25.4" y2="17.78" width="0.1524" layer="91"/>
+<wire x1="-25.4" y1="5.08" x2="-25.4" y2="7.62" width="0.1524" layer="91"/>
+<wire x1="-25.4" y1="7.62" x2="-25.4" y2="17.78" width="0.1524" layer="91"/>
 <wire x1="-25.4" y1="17.78" x2="-30.48" y2="17.78" width="0.1524" layer="91"/>
 <pinref part="JP1" gate="A" pin="1"/>
 <junction x="-30.48" y="17.78"/>
 <wire x1="-30.48" y1="17.78" x2="-33.02" y2="17.78" width="0.1524" layer="91"/>
+<pinref part="R6" gate="G$1" pin="1"/>
+<wire x1="-15.24" y1="7.62" x2="-20.32" y2="7.62" width="0.1524" layer="91"/>
+<junction x="-25.4" y="7.62"/>
+<pinref part="R5" gate="G$1" pin="1"/>
+<junction x="-20.32" y="7.62"/>
+<wire x1="-20.32" y1="7.62" x2="-25.4" y2="7.62" width="0.1524" layer="91"/>
 </segment>
 <segment>
@@
 </segment>
 </net>
-<net name="N$11" class="0">
+<net name="A=B" class="0">
 <segment>
 <wire x1="71.12" y1="99.06" x2="78.74" y2="99.06" width="0.1524" layer="91"/>
@@
 </segment>
 </net>
-<net name="RES" class="0">
+<net name="/RES" class="0">
 <segment>
 <wire x1="198.12" y1="48.26" x2="170.18" y2="48.26" width="0.1524" layer="91"/>
@@
 </segment>
 </net>
-<net name="DSR" class="0">
+<net name="/DSR" class="0">
 <segment>
 <pinref part="IC1" gate="G$1" pin="!DSR"/>
@@
 <junction x="20.32" y="7.62"/>
 <junction x="-7.62" y="25.4"/>
-<wire x1="-7.62" y1="25.4" x2="-33.02" y2="25.4" width="0.1524" layer="91"/>
-</segment>
-</net>
-<net name="DTR" class="0">
+<wire x1="-7.62" y1="25.4" x2="-20.32" y2="25.4" width="0.1524" layer="91"/>
+<pinref part="R5" gate="G$1" pin="2"/>
+<wire x1="-20.32" y1="25.4" x2="-33.02" y2="25.4" width="0.1524" layer="91"/>
+<wire x1="-20.32" y1="17.78" x2="-20.32" y2="25.4" width="0.1524" layer="91"/>
+<junction x="-20.32" y="25.4"/>
+</segment>
+</net>
+<net name="/DTR" class="0">
 <segment>
 <pinref part="IC1" gate="G$1" pin="!DTR"/>
@@
 </segment>
 </net>
-<net name="CTS" class="0">
+<net name="/CTS" class="0">
 <segment>
 <pinref part="IC1" gate="G$1" pin="!CTS"/>
@@
 <junction x="20.32" y="12.7"/>
 <junction x="-7.62" y="30.48"/>
-<wire x1="-7.62" y1="30.48" x2="-33.02" y2="30.48" width="0.1524" layer="91"/>
-</segment>
-</net>
-<net name="RTS" class="0">
+<wire x1="-7.62" y1="30.48" x2="-15.24" y2="30.48" width="0.1524" layer="91"/>
+<pinref part="R6" gate="G$1" pin="2"/>
+<wire x1="-15.24" y1="30.48" x2="-33.02" y2="30.48" width="0.1524" layer="91"/>
+<wire x1="-15.24" y1="17.78" x2="-15.24" y2="30.48" width="0.1524" layer="91"/>
+<junction x="-15.24" y="30.48"/>
+</segment>
+</net>
+<net name="/RTS" class="0">
 <segment>
 <pinref part="IC1" gate="G$1" pin="!RTS"/>
@@
 </segment>
 </net>
-<net name="N$6" class="0">
+<net name="-A=B" class="0">
 <segment>
 <pinref part="IC3" gate="C" pin="O"/>
@@
 </segment>
 </net>
-<net name="-RES" class="0">
+<net name="RES" class="0">
 <segment>
 <pinref part="7404" gate="B" pin="O"/>
